File: pcb/MGC_module.kicad_sch (KiCad schematic)
At the start: 52 parts, among them J11 103P012BB100, J12 103P012BB100, J13 103P012BB100, J3 103P012BB100, J7 103P012BB100, SW1 SW_DIP_x02, U1 74LVC4066, U2 74AHC1G14, U3 ATmega16A-A, Y1 12MHz

Commit message: Update uart series resistor values
Parts:
- R11, R12: value 0 -> 22k
Changed lines of the file:
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@@
 			)
 		)
-		(property "Value" "0"
-			(at 113.03 93.98 90)
+		(property "Value" "22k"
+			(at 109.22 99.06 90)
 			(effects
 				(font
@@
 			)
 		)
-		(property "Value" "0"
-			(at 115.57 93.98 90)
-			(effects
-				(font
+		(property "Value" "22k"
+			(at 116.84 99.06 90)
+			(effects
+				(font
