File: pcb/MGC_module.kicad_sch (KiCad schematic)
At the start: 52 parts, among them J11 103P012BB100, J12 103P012BB100, J13 103P012BB100, J3 103P012BB100, J7 103P012BB100, SW1 SW_DIP_x02, U1 74LVC4066, U2 74AHC1G14, U3 ATmega16A-A, Y1 12MHz

Commit message: Fix pwm resistor value
Parts:
- R10, R13, R14, R15, R16, R17, R19, R20, R21, R22, R6, R7, R8, R9: value 0 -> 0R
- R3: value 150 -> 10k; HTL 102934 -> 102967
Changed lines of the file:
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@@
 	(wire
 		(pts
-			(xy 111.76 88.9) (xy 111.76 95.25)
+			(xy 111.76 87.63) (xy 111.76 95.25)
 		)
 		(stroke
@@
 	(wire
 		(pts
-			(xy 114.3 88.9) (xy 114.3 95.25)
+			(xy 114.3 87.63) (xy 114.3 95.25)
 		)
 		(stroke
@@
 	)
 	(label "RXD"
-		(at 114.3 88.9 270)
+		(at 114.3 87.63 270)
 		(effects
 			(font
@@
 	)
 	(label "TXD"
-		(at 111.76 88.9 270)
+		(at 111.76 87.63 270)
 		(effects
 			(font
@@
 			)
 		)
-		(property "Value" "0"
+		(property "Value" "0R"
 			(at 207.01 132.08 90)
 			(effects
@@
 			)
 		)
-		(property "Value" "0"
+		(property "Value" "0R"
 			(at 243.84 121.92 90)
 			(effects
@@
 			)
 		)
-		(property "Value" "0"
+		(property "Value" "0R"
 			(at 157.48 114.3 90)
 			(effects
@@
 			)
 		)
-		(property "Value" "0"
+		(property "Value" "0R"
 			(at 157.48 137.16 90)
 			(effects
@@
 			)
 		)
-		(property "Value" "0"
+		(property "Value" "0R"
 			(at 243.84 127 90)
 			(effects
@@
 			)
 		)
-		(property "Value" "0"
+		(property "Value" "0R"
 			(at 231.14 132.08 90)
 			(effects
@@
 			)
 		)
-		(property "Value" "0"
+		(property "Value" "0R"
 			(at 271.78 127 90)
 			(effects
@@
 			)
 		)
-		(property "Value" "0"
+		(property "Value" "0R"
 			(at 243.84 132.08 90)
 			(effects
@@
 			)
 		)
-		(property "Value" "0"
+		(property "Value" "0R"
 			(at 160.02 118.11 90)
 			(effects
@@
 			)
 		)
-		(property "Value" "0"
-			(at 69.85 93.98 90)
+		(property "Value" "0R"
+			(at 67.31 93.98 90)
 			(effects
 				(font
@@
 		)
 		(property "Value" "22k"
-			(at 109.22 99.06 90)
+			(at 110.49 93.98 90)
 			(effects
 				(font
@@
 		)
 		(property "Value" "22k"
-			(at 116.84 99.06 90)
+			(at 113.03 93.98 90)
 			(effects
 				(font
@@
 			)
 		)
-		(property "Value" "0"
-			(at 90.17 93.98 90)
+		(property "Value" "0R"
+			(at 87.63 93.98 90)
 			(effects
 				(font
@@
 			)
 		)
-		(property "Value" "0"
-			(at 92.71 93.98 90)
+		(property "Value" "0R"
+			(at 90.17 93.98 90)
 			(effects
 				(font
@@
 			)
 		)
-		(property "Value" "150"
+		(property "Value" "10k"
 			(at 162.56 88.9 90)
 			(effects
@@
 			)
 		)
-		(property "HTL" "102934"
+		(property "HTL" "102967"
 			(at 162.56 86.36 90)
 			(effects
@@
 			)
 		)
-		(property "Value" "0"
+		(property "Value" "0R"
 			(at 160.02 125.73 90)
 			(effects
@@
 			)
 		)
-		(property "Value" "0"
-			(at 67.31 93.98 90)
+		(property "Value" "0R"
+			(at 64.77 93.98 90)
 			(effects
 				(font
