File: pcb/MGC_module.kicad_pcb (KiCad board)
At the start: 2 copper layers, 33 x 48.9 mm, 53 parts, among them J11 103P012BB100, J12 103P012BB100, J13 103P012BB100, J3 103P012BB100, J7 103P012BB100, SW1 SW_DIP_x02, U1 74LVC4066, U2 74AHC1G14, U3 ATmega16A-A, Y1 12MHz

Commit message: Fix pwm resistor value
Parts:
- R10, R13, R14, R15, R16, R17, R19, R20, R21, R22, R6, R7, R8, R9: value 0 -> 0R
- R3: value 150 -> 10k
Changed lines of the file:
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@@
 			)
 		)
-		(property "Value" "0"
+		(property "Value" "0R"
 			(at 2.54 0 90)
 			(layer "B.Fab")
@@
 			)
 		)
-		(property "Value" "0"
+		(property "Value" "0R"
 			(at -2.54 0 90)
 			(layer "B.Fab")
@@
 			)
 		)
-		(property "Value" "150"
+		(property "Value" "10k"
 			(at 0 -1.83 90)
 			(layer "B.Fab")
@@
 			)
 		)
-		(property "HTL" "102934"
+		(property "HTL" "102967"
 			(at 0 0 90)
 			(unlocked yes)
@@
 			)
 		)
-		(property "Value" "0"
+		(property "Value" "0R"
 			(at 2.54 0 90)
 			(layer "B.Fab")
@@
 			)
 		)
-		(property "Value" "0"
+		(property "Value" "0R"
 			(at 0 1.778 0)
 			(layer "B.Fab")
@@
 			)
 		)
-		(property "Value" "0"
+		(property "Value" "0R"
 			(at -2.54 0 90)
 			(layer "B.Fab")
@@
 			)
 		)
-		(property "Value" "0"
+		(property "Value" "0R"
 			(at 0 -1.83 0)
 			(layer "B.Fab")
@@
 			)
 		)
-		(property "Value" "0"
+		(property "Value" "0R"
 			(at -2.54 0 90)
 			(layer "B.Fab")
@@
 			)
 		)
-		(property "Value" "0"
+		(property "Value" "0R"
 			(at 0 -1.83 0)
 			(layer "B.Fab")
@@
 			)
 		)
-		(property "Value" "0"
+		(property "Value" "0R"
 			(at -2.54 0 90)
 			(layer "B.Fab")
@@
 			)
 		)
-		(property "Value" "0"
+		(property "Value" "0R"
 			(at 0 -1.83 90)
 			(layer "B.Fab")
@@
 			)
 		)
-		(property "Value" "0"
+		(property "Value" "0R"
 			(at 0 -1.83 90)
 			(layer "B.Fab")
@@
 			)
 		)
-		(property "Value" "0"
+		(property "Value" "0R"
 			(at -2.54 0 90)
 			(layer "B.Fab")
@@
 			)
 		)
-		(property "Value" "0"
+		(property "Value" "0R"
 			(at 2.54 0 90)
 			(layer "B.Fab")
@@
 			)
 		)
-		(property "Value" "0"
+		(property "Value" "0R"
 			(at -2.54 0 90)
 			(layer "B.Fab")
